Commit message: Configured tested world and robot visuals using Rviz and Gazebo

File: src/warehouse_robot/urdf/robot.urdf.xacro (robot description, xacro)
@@ -7,5 +7,11 @@
   <xacro:property name="wheel_radius" value="0.08"/>
   <xacro:property name="wheel_width" value="0.05"/>
-  <xacro:property name="wheel_separation" value="0.4"/>
+  <xacro:property name="wheel_separation" value="0.40"/>
+  <!-- ================= ROOT LINK ================= -->
+  <link name="world"/>
+  <joint name="world_to_base" type="fixed">
+    <parent link="world"/>
+    <child link="base_link"/>
+  </joint>
   <!-- ================= BASE ================= -->
   <link name="base_link">
@@ -14,6 +20,24 @@
         <box size="${base_length} ${base_width} ${base_height}"/>
       </geometry>
-      <material name="blue">
-        <color rgba="0.2 0.2 0.8 1"/>
+      <material name="yellow">
+        <color rgba="1.0 0.85 0.0 1.0"/>
+      </material>
+    </visual>
+    <visual>
+      <origin xyz="0 0 ${base_height/2 + 0.008}" rpy="0 0 0"/>
+      <geometry>
+        <box size="${base_length*0.88} ${base_width*0.82} 0.015"/>
+      </geometry>
+      <material name="top_panel_dark">
+        <color rgba="0.18 0.18 0.18 1.0"/>
+      </material>
+    </visual>
+    <visual>
+      <origin xyz="${base_length/2 - 0.006} 0 0" rpy="0 0 0"/>
+      <geometry>
+        <box size="0.012 ${base_width*0.72} ${base_height*0.45}"/>
+      </geometry>
+      <material name="front_accent_cyan">
+        <color rgba="0.0 0.85 1.0 1.0"/>
       </material>
     </visual>
@@ -24,8 +48,8 @@
     </collision>
     <inertial>
-      <mass value="10.0"/>
-      <inertia ixx="0.5" ixy="0" ixz="0"
-               iyy="0.5" iyz="0"
-               izz="0.5"/>
+      <mass value="8.0"/>
+      <inertia ixx="0.2" ixy="0" ixz="0"
+               iyy="0.2" iyz="0"
+               izz="0.2"/>
     </inertial>
   </link>
@@ -36,11 +60,25 @@
         <cylinder radius="${wheel_radius}" length="${wheel_width}"/>
       </geometry>
+      <material name="black">
+        <color rgba="0 0 0 1"/>
+      </material>
     </visual>
+    <collision>
+      <geometry>
+        <cylinder radius="${wheel_radius}" length="${wheel_width}"/>
+      </geometry>
+    </collision>
+    <inertial>
+      <mass value="1.0"/>
+      <inertia ixx="0.01" ixy="0" ixz="0"
+               iyy="0.01" iyz="0"
+               izz="0.01"/>
+    </inertial>
   </link>
   <joint name="left_wheel_joint" type="continuous">
     <parent link="base_link"/>
     <child link="left_wheel"/>
-    <origin xyz="0 ${wheel_separation/2} -0.1" rpy="0 1.5707 0"/>
-    <axis xyz="0 0 1"/>
+    <origin xyz="0 ${wheel_separation/2} -${base_height/2}" rpy="1.5707 0 0"/>
+    <axis xyz="0 1 0"/>
   </joint>
   <!-- ================= RIGHT WHEEL ================= -->
@@ -50,13 +88,27 @@
         <cylinder radius="${wheel_radius}" length="${wheel_width}"/>
       </geometry>
+      <material name="black">
+        <color rgba="0 0 0 1"/>
+      </material>
     </visual>
+    <collision>
+      <geometry>
+        <cylinder radius="${wheel_radius}" length="${wheel_width}"/>
+      </geometry>
+    </collision>
+    <inertial>
+      <mass value="1.0"/>
+      <inertia ixx="0.01" ixy="0" ixz="0"
+               iyy="0.01" iyz="0"
+               izz="0.01"/>
+    </inertial>
   </link>
   <joint name="right_wheel_joint" type="continuous">
     <parent link="base_link"/>
     <child link="right_wheel"/>
-    <origin xyz="0 -${wheel_separation/2} -0.1" rpy="0 1.5707 0"/>
-    <axis xyz="0 0 1"/>
+    <origin xyz="0 -${wheel_separation/2} -${base_height/2}" rpy="1.5707 0 0"/>
+    <axis xyz="0 1 0"/>
   </joint>
-  <!-- ================= CASTER ================= -->
+  <!-- ================= CASTER WHEEL ================= -->
   <link name="caster_wheel">
     <visual>
@@ -64,4 +116,7 @@
         <sphere radius="0.05"/>
       </geometry>
+      <material name="gray">
+        <color rgba="0.5 0.5 0.5 1"/>
+      </material>
     </visual>
   </link>
@@ -69,5 +124,5 @@
     <parent link="base_link"/>
     <child link="caster_wheel"/>
-    <origin xyz="-0.2 0 -0.1"/>
+    <origin xyz="-0.2 0 -${base_height/2}"/>
   </joint>
   <!-- ================= LIDAR ================= -->
@@ -75,8 +130,17 @@
     <visual>
       <geometry>
-        <cylinder radius="0.05" length="0.05"/>
+        <cylinder radius="0.045" length="0.04"/>
       </geometry>
-      <material name="black">
-        <color rgba="0 0 0 1"/>
+      <material name="lidar_body">
+        <color rgba="0.10 0.10 0.12 1.0"/>
+      </material>
+    </visual>
+    <visual>
+      <origin xyz="0 0 0.022" rpy="0 0 0"/>
+      <geometry>
+        <cylinder radius="0.028" length="0.010"/>
+      </geometry>
+      <material name="lidar_glow">
+        <color rgba="0.0 0.95 1.0 1.0"/>
       </material>
     </visual>
@@ -85,9 +149,9 @@
     <parent link="base_link"/>
     <child link="laser_frame"/>
-    <origin xyz="0.2 0 0.15"/>
+    <origin xyz="0.2 0 ${base_height/2 + 0.025}"/>
   </joint>
   <!-- ================= GAZEBO: DIFF DRIVE ================= -->
   <gazebo>
-    <plugin name="gz::sim::systems::DiffDrive" filename="gz-sim-diff-drive-system">
+    <plugin name="diff_drive" filename="gz-sim-diff-drive-system">
       <left_joint>left_wheel_joint</left_joint>
       <right_joint>right_wheel_joint</right_joint>

Commit message: fix robot spawn position and adjust URDF for movement issues

File: src/warehouse_robot/urdf/robot.urdf.xacro (robot description, xacro)
@@ -8,10 +8,4 @@
   <xacro:property name="wheel_width" value="0.05"/>
   <xacro:property name="wheel_separation" value="0.40"/>
-  <!-- ================= ROOT LINK ================= -->
-  <link name="world"/>
-  <joint name="world_to_base" type="fixed">
-    <parent link="world"/>
-    <child link="base_link"/>
-  </joint>
   <!-- ================= BASE ================= -->
   <link name="base_link">
@@ -163,4 +157,6 @@
       <frame_id>odom</frame_id>
       <child_frame_id>base_link</child_frame_id>
+      <publish_odom>true</publish_odom>
+      <publish_tf>true</publish_tf>
     </plugin>
   </gazebo>

Commit message: Fixed and completed mapping and localization

File: src/warehouse_robot/urdf/robot.urdf.xacro (robot description, xacro)
@@ -8,5 +8,8 @@
   <xacro:property name="wheel_width" value="0.05"/>
   <xacro:property name="wheel_separation" value="0.40"/>
-  <!-- ================= BASE ================= -->
+  <!-- ================= BASE (root link) =================
+       NOTE: base_link is the ROOT of the kinematic tree.
+       Do NOT anchor it to a "world" link with a fixed joint —
+       that would pin the robot at the origin and break odom/TF. -->
   <link name="base_link">
     <visual>
@@ -48,70 +51,114 @@
     </inertial>
   </link>
-  <!-- ================= LEFT WHEEL ================= -->
-  <link name="left_wheel">
-    <visual>
-      <geometry>
-        <cylinder radius="${wheel_radius}" length="${wheel_width}"/>
-      </geometry>
-      <material name="black">
-        <color rgba="0 0 0 1"/>
+  <!-- ================= WHEEL MACRO =================
+       Orientation note: the cylinder is lying on its side via rpy=(π/2, 0, 0),
+       so the cylinder's *length* axis (its local Z) now points along the
+       parent's Y axis (the axle direction).
+       The JOINT AXIS must therefore be (0 0 1) — i.e. the child's Z axis —
+       so the wheel rotates about its axle. The previous (0 1 0) made the
+       child's Y the rotation axis, which maps to the parent's Z (vertical),
+       causing the wheel to spin like a top and scrub sideways.          -->
+  <xacro:macro name="drive_wheel" params="side y_sign">
+    <link name="${side}_wheel">
+      <!-- Tyre -->
+      <visual>
+        <geometry>
+          <cylinder radius="${wheel_radius}" length="${wheel_width}"/>
+        </geometry>
+        <material name="tyre_black">
+          <color rgba="0.05 0.05 0.05 1"/>
+        </material>
+      </visual>
+      <!-- Hub (bright disk) so we can see the wheel rotate -->
+      <visual>
+        <origin xyz="0 0 ${wheel_width/2 + 0.001}" rpy="0 0 0"/>
+        <geometry>
+          <cylinder radius="${wheel_radius*0.45}" length="0.004"/>
+        </geometry>
+        <material name="wheel_hub">
+          <color rgba="0.85 0.85 0.90 1"/>
+        </material>
+      </visual>
+      <!-- Spoke 1: asymmetric stripe from hub to rim. Because the cylinder's
+           local Z is the axle direction, a box offset along local X rotates
+           visibly around the axle as the joint spins. -->
+      <visual>
+        <origin xyz="${wheel_radius*0.6} 0 ${wheel_width/2 + 0.002}" rpy="0 0 0"/>
+        <geometry>
+          <box size="${wheel_radius*0.7} 0.012 0.006"/>
+        </geometry>
+        <material name="spoke_cyan">
+          <color rgba="0.0 0.85 1.0 1.0"/>
+        </material>
+      </visual>
+      <!-- Spoke 2: perpendicular, different colour -->
+      <visual>
+        <origin xyz="0 ${wheel_radius*0.6} ${wheel_width/2 + 0.002}" rpy="0 0 0"/>
+        <geometry>
+          <box size="0.012 ${wheel_radius*0.7} 0.006"/>
+        </geometry>
+        <material name="spoke_yellow">
+          <color rgba="1.0 0.85 0.0 1.0"/>
+        </material>
+      </visual>
+      <collision>
+        <geometry>
+          <cylinder radius="${wheel_radius}" length="${wheel_width}"/>
+        </geometry>
+      </collision>
+      <inertial>
+        <mass value="1.0"/>
+        <inertia ixx="0.01" ixy="0" ixz="0"
+                 iyy="0.01" iyz="0"
+                 izz="0.01"/>
+      </inertial>
+    </link>
+    <joint name="${side}_wheel_joint" type="continuous">
+      <parent link="base_link"/>
+      <child link="${side}_wheel"/>
+      <origin xyz="0 ${y_sign*wheel_separation/2} -${base_height/2}" rpy="1.5707 0 0"/>
+      <!-- Axle axis (child Z == parent Y after the rpy rotation above) -->
+      <axis xyz="0 0 1"/>
+      <dynamics damping="0.01" friction="0.0"/>
+    </joint>
+    <!-- Good rolling friction for wheels -->
+    <gazebo reference="${side}_wheel">
+      <mu1>1.0</mu1>
+      <mu2>1.0</mu2>
+      <kp>1000000.0</kp>
+      <kd>100.0</kd>
+    </gazebo>
+  </xacro:macro>
+  <xacro:drive_wheel side="left"  y_sign="1"/>
+  <xacro:drive_wheel side="right" y_sign="-1"/>
+  <!-- ================= CASTER WHEEL ================= -->
+  <link name="caster_wheel">
+    <visual>
+      <geometry>
+        <sphere radius="0.05"/>
+      </geometry>
+      <material name="gray">
+        <color rgba="0.5 0.5 0.5 1"/>
       </material>
     </visual>
     <collision>
       <geometry>
-        <cylinder radius="${wheel_radius}" length="${wheel_width}"/>
-      </geometry>
+        <sphere radius="0.05"/>
+      </geometry>
+      <surface>
+        <friction>
+          <ode>
+            <mu>0.0</mu>
+            <mu2>0.0</mu2>
+          </ode>
+        </friction>
+      </surface>
     </collision>
     <inertial>
-      <mass value="1.0"/>
-      <inertia ixx="0.01" ixy="0" ixz="0"
-               iyy="0.01" iyz="0"
-               izz="0.01"/>
+      <mass value="0.2"/>
+      <inertia ixx="0.0005" ixy="0" ixz="0"
+               iyy="0.0005" iyz="0"
+               izz="0.0005"/>
     </inertial>
-  </link>
-  <joint name="left_wheel_joint" type="continuous">
-    <parent link="base_link"/>
-    <child link="left_wheel"/>
-    <origin xyz="0 ${wheel_separation/2} -${base_height/2}" rpy="1.5707 0 0"/>
-    <axis xyz="0 1 0"/>
-  </joint>
-  <!-- ================= RIGHT WHEEL ================= -->
-  <link name="right_wheel">
-    <visual>
-      <geometry>
-        <cylinder radius="${wheel_radius}" length="${wheel_width}"/>
-      </geometry>
-      <material name="black">
-        <color rgba="0 0 0 1"/>
-      </material>
-    </visual>
-    <collision>
-      <geometry>
-        <cylinder radius="${wheel_radius}" length="${wheel_width}"/>
-      </geometry>
-    </collision>
-    <inertial>
-      <mass value="1.0"/>
-      <inertia ixx="0.01" ixy="0" ixz="0"
-               iyy="0.01" iyz="0"
-               izz="0.01"/>
-    </inertial>
-  </link>
-  <joint name="right_wheel_joint" type="continuous">
-    <parent link="base_link"/>
-    <child link="right_wheel"/>
-    <origin xyz="0 -${wheel_separation/2} -${base_height/2}" rpy="1.5707 0 0"/>
-    <axis xyz="0 1 0"/>
-  </joint>
-  <!-- ================= CASTER WHEEL ================= -->
-  <link name="caster_wheel">
-    <visual>
-      <geometry>
-        <sphere radius="0.05"/>
-      </geometry>
-      <material name="gray">
-        <color rgba="0.5 0.5 0.5 1"/>
-      </material>
-    </visual>
   </link>
   <joint name="caster_joint" type="fixed">
@@ -120,4 +167,9 @@
     <origin xyz="-0.2 0 -${base_height/2}"/>
   </joint>
+  <!-- Low-friction caster surface for Gazebo -->
+  <gazebo reference="caster_wheel">
+    <mu1>0.0</mu1>
+    <mu2>0.0</mu2>
+  </gazebo>
   <!-- ================= LIDAR ================= -->
   <link name="laser_frame">
@@ -139,4 +191,15 @@
       </material>
     </visual>
+    <collision>
+      <geometry>
+        <cylinder radius="0.045" length="0.04"/>
+      </geometry>
+    </collision>
+    <inertial>
+      <mass value="0.1"/>
+      <inertia ixx="0.0001" ixy="0" ixz="0"
+               iyy="0.0001" iyz="0"
+               izz="0.0001"/>
+    </inertial>
   </link>
   <joint name="laser_joint" type="fixed">
@@ -145,7 +208,13 @@
     <origin xyz="0.2 0 ${base_height/2 + 0.025}"/>
   </joint>
-  <!-- ================= GAZEBO: DIFF DRIVE ================= -->
+  <!-- ================= GAZEBO: DIFF DRIVE =================
+       Publishes:
+         - Reads  geometry_msgs/Twist on gz topic  /cmd_vel
+         - Writes nav_msgs/Odometry   on gz topic  /odom
+         - Writes TF (Pose_V)         on gz topic  /tf
+         These are bridged to ROS in the launch file. -->
   <gazebo>
-    <plugin name="gz::sim::systems::DiffDrive" filename="gz-sim-diff-drive-system">
+    <plugin filename="gz-sim-diff-drive-system"
+            name="gz::sim::systems::DiffDrive">
       <left_joint>left_wheel_joint</left_joint>
       <right_joint>right_wheel_joint</right_joint>
@@ -155,8 +224,17 @@
       <topic>/cmd_vel</topic>
       <odom_topic>/odom</odom_topic>
+      <tf_topic>/tf</tf_topic>
       <frame_id>odom</frame_id>
       <child_frame_id>base_link</child_frame_id>
-      <publish_odom>true</publish_odom>
-      <publish_tf>true</publish_tf>
+      <!-- Sane accel/velocity limits so the bot doesn't rocket off -->
+      <max_linear_acceleration>2.0</max_linear_acceleration>
+      <max_angular_acceleration>4.0</max_angular_acceleration>
+    </plugin>
+    <!-- Publishes simulation time on gz topic /clock -->
+    <plugin filename="gz-sim-joint-state-publisher-system"
+            name="gz::sim::systems::JointStatePublisher">
+      <topic>/joint_states</topic>
+      <joint_name>left_wheel_joint</joint_name>
+      <joint_name>right_wheel_joint</joint_name>
     </plugin>
   </gazebo>
@@ -166,4 +244,5 @@
       <update_rate>10</update_rate>
       <topic>/scan</topic>
+      <gz_frame_id>laser_frame</gz_frame_id>
       <lidar>
         <scan>
